File: hardware/limelight.kicad_pcb (KiCad board)
At the start: 2 copper layers, 49.5 x 51.5 mm, 21 parts, among them J1 +5V IN, J2 DMG1083 Panel Output, SW1 SW1, SW2 SW2, SW3 RESET, U1 Pico, U4 74HCT245, U5 74HCT245, U6 74HCT245

Commit message: Finish PCB ready for fab
Parts:
- added D3: PWR, LED_SMD:LED_0603_1608Metric, F.Cu at (147.6, 110.6)
- added R4: 1k, Resistor_SMD:R_0603_1608Metric, F.Cu at (144.4, 110.6)
- D1: value LED -> LED1
- D2: value LED -> LED2
- J1: value +5V IN -> +5V GND
- R1: value 4.7k -> 10k
- R8, R9: footprint Resistor_SMD:R_0402_1005Metric -> Resistor_SMD:R_0603_1608Metric
- U1: value Pico -> Pi Pico WH
- moved R1 21.4 mm to (150.7, 74.6), turned to 180 degrees
- moved R2 10.6 mm to (159.4, 67.8), turned to 90 degrees
- moved D2 6.11 mm to (147.6, 114.2), turned to 180 degrees
- moved R5 4.11 mm to (158.2, 67.8), turned to 90 degrees
- moved R3 3.42 mm to (140.2, 66.9), turned to -90 degrees
- moved R8 3.24 mm to (144.4, 112.4)
- moved R9 2.94 mm to (144.4, 114.2)
- moved D1 2.82 mm to (147.6, 112.4), turned to 180 degrees
- moved D4 2.37 mm to (155.6, 111.6), turned to -90 degrees
- turned C8 to 0 degrees
Routing:
- net +3V3: track 0.00 -> 100.0 mm, vias 0 -> 2
- net /LED2: track 0.00 -> 81.7 mm, vias 0 -> 1
- net /nSHIFT_EN: track 0.00 -> 63.3 mm, vias 0 -> 1
- net /RUN: track 0.00 -> 54.0 mm, vias 0 -> 1
- net /R2_3V3: track 0.00 -> 43.7 mm, vias 0 -> 1
- net /SW2: track 0.00 -> 42.4 mm, vias 0 -> 1
- net /B2_3V3: track 0.00 -> 40.9 mm
- net /G1_3V3: track 0.00 -> 40.5 mm, vias 0 -> 1
- net /G2_3V3: track 0.00 -> 39.7 mm
- net /B1_3V3: track 0.00 -> 34.3 mm
- net /R1_3V3: track 0.00 -> 33.7 mm
- net /LAT_3V3: track 0.00 -> 32.9 mm
- net /DCLK_3V3: track 0.00 -> 32.6 mm, vias 0 -> 1
- net /ADDR_E_3V3: track 0.00 -> 31.7 mm, vias 0 -> 1
- net /R3_3V3: track 0.00 -> 31.3 mm, vias 0 -> 1
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- added copper zone on In2.Cu, net +5V
- added copper zone on In1.Cu, net GND
Other:
- copper layers 2 -> 4
- board text added: "1"
- board text added: "DAVID TURNER JUNE 2024 github.com/cillian64/limelight"
- board text added: "LIMELIGHT r1"
- board text added: "RST"

Commit message: Files sent to production
Parts:
- added J3: Barrel_Jack, Connector_BarrelJack:BarrelJack_Horizontal, F.Cu at (151.8, 111.7)
- added REF**: Symbol_Barrel_Polarity, Symbol:Symbol_Barrel_Polarity, B.Cu at (155.2, 115.0)
- J1: value +5V GND -> +5V IN; footprint Connector_PinHeader_2.54mm:PinHeader_1x02_P2.54mm_Vertical -> Connector_Wire:SolderWire-2.5sqmm_1x02_P8.8mm_D2.4mm_OD4.4mm
- U1: value Pi Pico WH -> Pi Pico
- moved D4 9.70 mm to (146.2, 109.2), turned to 0 degrees
- moved R5 8.22 mm to (153.9, 74.8), turned to 180 degrees
- moved R2 7.87 mm to (155.8, 74.8), turned to 0 degrees
- moved C10 6.50 mm to (152.5, 96.2)
- moved J2 5.84 mm to (160.6, 66.9)
- moved C8 5.57 mm to (151.6, 74.9), turned to 180 degrees
- moved C9 5.23 mm to (151.2, 85.0), turned to 180 degrees
- moved D3 1.40 mm to (147.7, 112.0)
- moved R4 1.40 mm to (144.5, 112.0)
- moved D1 1.40 mm to (147.7, 113.8)
- moved D2 1.40 mm to (147.7, 115.6)
- moved R8 1.40 mm to (144.5, 113.8)
- moved R9 1.40 mm to (144.5, 115.6)
- moved R1 1.01 mm to (149.7, 74.8)
- moved J1 0.55 mm to (162.3, 113.2), turned to 90 degrees
Routing:
- net /+5V_IN: track 4.68 -> 92.6 mm
- net GND: track 30.0 -> 46.4 mm, vias 11 -> 13
- net +3V3: track 100.0 -> 84.2 mm, vias 2 -> 3
- net /RUN: track 54.0 -> 43.8 mm
- net /SW2: track 42.4 -> 48.9 mm
- net /GCLK: track 9.80 -> 14.0 mm
- net /ADDR_B: track 12.3 -> 16.3 mm
- net /ADDR_A: track 9.51 -> 13.5 mm
- net /DCLK: track 9.02 -> 12.6 mm
- net /LAT: track 14.0 -> 17.5 mm
- net /R1: track 12.0 -> 14.5 mm
- net /B3: track 8.94 -> 11.5 mm
- net /G1: track 8.66 -> 11.2 mm
- net /B1: track 11.8 -> 14.0 mm
- net /R4: track 9.07 -> 10.7 mm
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Other:
- board text added: "+"
- board text added: "+5V"
- board text added: "-"
- board text added: "David Turner Feb 2025 github.com/cillian64/limelight"
- board text added: "JLCJLCJLCJLC"
- board text removed: "DAVID TURNER JUNE 2024 github.com/cillian64/limelight"
